Commit message: update for cluster distributed running

File: source/whole_body_tracking/whole_body_tracking/tasks/tracking/empty_proxy.urdf (robot description, URDF)
Before this commit: robot empty_proxy, 1 links, 0 joints
Links:
- link proxy_base: mass None -> 0.001; geometry collision box size=0.001 0.001 0.001; visual box size=0.001 0.001 0.001
